File: Hummingbird/teensy.sch (KiCad schematic (older format))
At the start: 0 parts

Commit message: Update (?)
Parts:
- added U?: Teensy3.2, symbol teensy:Teensy3.2
Changed lines of the file:
@@
 $Descr A4 11693 8268
 encoding utf-8
-Sheet 1 9
+Sheet 5 10
 Title ""
 Date ""
@@
 Comment4 ""
 $EndDescr
+$Comp
+L teensy:Teensy3.2 U?
+U 1 1 60BFBCAE
+P 5650 3650
+F 0 "U?" H 5650 5287 60  0000 C CNN
+F 1 "Teensy3.2" H 5650 5181 60  0000 C CNN
+F 2 "" H 5650 2900 60  0000 C CNN
+F 3 "" H 5650 2900 60  0000 C CNN
+	1    5650 3650
+	1    0    0    -1
+$EndComp
 $EndSCHEMATC
